Commit message: feat: 更新机械臂urdf文件

File: web/public/3dModules/roboticArm.urdf (robot description, URDF)
Before this commit: robot robotic_arm, 6 links, 5 joints
Links:
- removed link base_link
- added link link_0; visual mesh filename=link0.STL
- link link_1: geometry visual mesh filename=link1.STL
- link link_2: geometry visual mesh filename=link2.STL
- link link_3: geometry visual mesh filename=link3.STL
- link link_4: geometry visual mesh filename=link4.STL
- link link_5: geometry visual mesh filename=link5.STL
Joints:
- joint joint_1: parent base_link -> link_0
